File: hardware/ride_on/ride_on.kicad_sch (KiCad schematic)
At the start: 23 parts, among them J1 LCD_Module, J2 MicroSD_Module, U1 ESP32-S3-WROOM-1, U2 MAX98357A Module, U3 SN74AHCT125N, U4 MP1584EN Buck Module, U5 MP1584EN Buck Module, U6 MAX98357A Module

Commit message: save current schematic
Parts:
- removed BT1: HY2005RX-24V40A, symbol Device:Battery
- removed C2: 1000uF 6V3+, symbol Device:C_Polarized
- removed D3, D4: WS2812B, LED_SMD:LED_WS2812B_PLCC4_5.0x5.0mm_P3.2mm, symbol LED:WS2812B
- added J3: 24V Battery, symbol Connector_Generic:Conn_01x02
- added R7, R8: 330R, symbol Device:R_Small_US
- C1: value 1000uF 6V3+ -> 1000uF
Connections:
- net AMP_BCLK: no longer U6.16 (BCLK)
- net AMP_DIN: no longer U6.1 (DIN)
- net AMP_LRC: no longer U6.14 (LRC)
- net GNDREF: now also J1.13 (GND), J2.6 (GND), J3.2 (Pin_2)
- net +24V: now reaches U4.1 (V_{IN}+), U5.1 (V_{IN}+)
- net +24V: now also J3.1 (Pin_1)
- net +5VA: now reaches U1.1 (5V_{IN}), U4.4 (V_{OUT}+)
- net +5VA: now also J1.14 (VCC), J2.5 (VCC)
- net +3V3: now reaches R3.1, R4.1, R5.1, R6.1, U1.2 (GND)
- net BODYLIGHT_L_OE_GPIO39: now reaches R4.2, U3.10 (3~{OE})
- net BODYLIGHT_L_OE_GPIO39: now also U1.23 (GPIO39)
- net at D1.4 (DIN): no longer R1.2
- net HEADLIGHT_R_DC_GPIO42: now reaches R2.2
- net HEADLIGHT_R_DC_GPIO42: now also U1.14 (GPIO41), U3.5 (2A)
- net at C1.1, D1.1 (VDD), D2.1 (VDD): no longer U3.14 (VCC), U5.4 (V_{OUT}+)
- net HEADLIGHT_L_OE_GPIO1: now reaches R6.2, U1.10 (GPIO1), U3.1 (1~{OE})
- net HEADLIGHT_L_DC_GPIO2: now reaches U1.11 (GPIO2), U3.2 (1A)
- net HEADLIGHT_L_DC_GPIO2: now also R1.2
- net HEADLIGHT_R_OE_GPIO41: now reaches R3.2, U1.13 (GPIO42), U3.4 (2~{OE})
- net BODYLIGHT_L_DC_GPIO38: now reaches U1.28 (GPIO38)
- net BODYLIGHT_L_DC_GPIO38: now also U3.9 (3A), R7.2
- net BODYLIGHT_R_OE_GPIO37: now reaches U1.29 (GPIO37)
- net BODYLIGHT_R_OE_GPIO37: now also R5.2, U3.13 (4~{OE})
- net BODYLIGHT_R_DC_GPIO36: now reaches U1.30 (GPIO36)
- net BODYLIGHT_R_DC_GPIO36: now also U3.12 (4A), R8.2
- net at U3.11 (4Y): now also R8.1
- net at U3.8 (3Y): now also R7.1
- new net +5VB: U3.14 (VCC), U5.4 (V_{OUT}+)
- no-connect marks 11 -> 16
Other:
- note removed: "5v tolerant"
- moved on the sheet: C1, D1, D2, J1, J2, LS1, LS2, R3, R4, R5, R6, U1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
